File: apple_update/schematics/Connectors.sch (KiCad schematic (older format))
At the start: 5 parts, among them J401 Conn_01x06, SW401 SW_DIP_x08

Commit message: Update labels
Parts:
- removed R401: R, symbol Device:R
Changed lines of the file:
@@
-$EndComp
-$Comp
-L Device:R R?
-U 1 1 653122D2
-P 4500 2800
-AR Path="/653122D2" Ref="R?"  Part="1"
-AR Path="/652C7050/653122D2" Ref="R401"  Part="1"
-F 0 "R401" H 4650 2750 50  0000 R CNN
-F 1 "R" H 4650 2850 50  0000 R CNN
-F 2 "" V 4430 2800 50  0001 C CNN
-F 3 "~" H 4500 2800 50  0001 C CNN
-	1    4500 2800
-	-1   0    0    1
-$EndComp
-$Comp
-L power:+3V3 #PWR?
-U 1 1 653122D8
-P 4500 2500
-AR Path="/653122D8" Ref="#PWR?"  Part="1"
-AR Path="/652C7050/653122D8" Ref="#PWR0401"  Part="1"
-F 0 "#PWR0401" H 4500 2350 50  0001 C CNN
-F 1 "+3V3" H 4515 2673 50  0000 C CNN
-F 2 "" H 4500 2500 50  0001 C CNN
-F 3 "" H 4500 2500 50  0001 C CNN
-	1    4500 2500
-	1    0    0    -1
 $EndComp
 $Comp
@@
 	5450 2600 5450 3250
 Wire Wire Line
-	4500 2650 4500 2500
-Wire Wire Line
-	4500 2950 4500 3250
-Wire Wire Line
-	4500 3250 4750 3250
-Wire Wire Line
 	4750 2950 4750 3250
 Connection ~ 4750 3250
 Wire Wire Line
 	4750 3250 4800 3250
-Connection ~ 4500 3250
 $Comp
 L power:+3V3 #PWR?
@@
 Wire Wire Line
 	3950 3950 4650 3950
-Wire Wire Line
-	3950 3250 4500 3250
 Text HLabel 6350 2750 0    50   Input ~ 0
 SWDIO
@@
 Text Label 6450 3350 0    50   ~ 0
 VB
+Wire Wire Line
+	3950 3250 4750 3250
 $EndSCHEMATC

Commit message: updating sch. adding footprint for alps.
Parts:
- C401: footprint (none) -> Capacitor_SMD:C_0805_2012Metric_Pad1.18x1.45mm_HandSolder
- J401: footprint (none) -> Connector_PinHeader_1.00mm:PinHeader_1x06_P1.00mm_Horizontal
- R402: footprint (none) -> Resistor_SMD:R_0805_2012Metric_Pad1.20x1.40mm_HandSolder
- SW401: footprint (none) -> Button_Switch_THT:SW_DIP_SPSTx08_Slide_6.7x21.88mm_W7.62mm_P2.54mm_LowProfile
Changed lines of the file:
@@
 F 0 "SW401" H 5100 4317 50  0000 C CNN
 F 1 "SW_DIP_x08" H 5100 4226 50  0000 C CNN
-F 2 "" H 5100 3650 50  0001 C CNN
+F 2 "Button_Switch_THT:SW_DIP_SPSTx08_Slide_6.7x21.88mm_W7.62mm_P2.54mm_LowProfile" H 5100 3650 50  0001 C CNN
 F 3 "~" H 5100 3650 50  0001 C CNN
 	1    5100 3650
@@
 F 0 "C401" H 4635 2754 50  0000 R CNN
 F 1 "100nF" H 4635 2845 50  0000 R CNN
-F 2 "" H 4788 2650 50  0001 C CNN
+F 2 "Capacitor_SMD:C_0805_2012Metric_Pad1.18x1.45mm_HandSolder" H 4788 2650 50  0001 C CNN
 F 3 "~" H 4750 2800 50  0001 C CNN
 	1    4750 2800
@@
 F 0 "R402" H 4720 4246 50  0000 L CNN
 F 1 "10K" H 4720 4155 50  0000 L CNN
-F 2 "" V 4580 4200 50  0001 C CNN
+F 2 "Resistor_SMD:R_0805_2012Metric_Pad1.20x1.40mm_HandSolder" V 4580 4200 50  0001 C CNN
 F 3 "~" H 4650 4200 50  0001 C CNN
 	1    4650 4200
@@
 F 0 "J401" H 7180 2842 50  0000 L CNN
 F 1 "Conn_01x06" H 7180 2751 50  0000 L CNN
-F 2 "" H 7100 2850 50  0001 C CNN
+F 2 "Connector_PinHeader_1.00mm:PinHeader_1x06_P1.00mm_Horizontal" H 7100 2850 50  0001 C CNN
 F 3 "~" H 7100 2850 50  0001 C CNN
 	1    7100 2850
