File: apple_update/schematics/STM32.sch (KiCad schematic (older format))
At the start: 3 parts

Commit message: Update labels
Parts:
- gave numbers to parts that had none: 3
Other:
- moved on the sheet: L101
Changed lines of the file:
@@
 P 5700 3300
 AR Path="/652FE508" Ref="U?"  Part="1"
-AR Path="/652C6908/652FE508" Ref="U?"  Part="1"
-F 0 "U?" V 6250 4050 50  0000 C CNN
+AR Path="/652C6908/652FE508" Ref="U101"  Part="1"
+F 0 "U101" V 6250 4050 50  0000 C CNN
 F 1 "STM32F401CCUx" V 6250 4450 50  0000 C CNN
 F 2 "Package_DFN_QFN:QFN-48-1EP_7x7mm_P0.5mm_EP5.6x5.6mm" H 5100 1800 50  0001 R CNN
@@
 P 5700 1550
 AR Path="/652FE510" Ref="#PWR?"  Part="1"
-AR Path="/652C6908/652FE510" Ref="#PWR?"  Part="1"
-F 0 "#PWR?" H 5700 1400 50  0001 C CNN
+AR Path="/652C6908/652FE510" Ref="#PWR0104"  Part="1"
+F 0 "#PWR0104" H 5700 1400 50  0001 C CNN
 F 1 "+3V3" H 5715 1723 50  0000 C CNN
 F 2 "" H 5700 1550 50  0001 C CNN
@@
 P 5700 5050
 AR Path="/652FE51D" Ref="#PWR?"  Part="1"
-AR Path="/652C6908/652FE51D" Ref="#PWR?"  Part="1"
-F 0 "#PWR?" H 5700 4800 50  0001 C CNN
+AR Path="/652C6908/652FE51D" Ref="#PWR0105"  Part="1"
+F 0 "#PWR0105" H 5700 4800 50  0001 C CNN
 F 1 "GND" H 5705 4877 50  0000 C CNN
 F 2 "" H 5700 5050 50  0001 C CNN
@@
 P 5500 5050
 AR Path="/652FE523" Ref="#PWR?"  Part="1"
-AR Path="/652C6908/652FE523" Ref="#PWR?"  Part="1"
-F 0 "#PWR?" H 5500 4800 50  0001 C CNN
+AR Path="/652C6908/652FE523" Ref="#PWR0103"  Part="1"
+F 0 "#PWR0103" H 5500 4800 50  0001 C CNN
 F 1 "GND" H 5505 4877 50  0000 C CNN
 F 2 "" H 5500 5050 50  0001 C CNN
@@
 P 5900 5050
 AR Path="/652FE529" Ref="#PWR?"  Part="1"
-AR Path="/652C6908/652FE529" Ref="#PWR?"  Part="1"
-F 0 "#PWR?" H 5900 4800 50  0001 C CNN
+AR Path="/652C6908/652FE529" Ref="#PWR0106"  Part="1"
+F 0 "#PWR0106" H 5900 4800 50  0001 C CNN
 F 1 "GND" H 5905 4877 50  0000 C CNN
 F 2 "" H 5900 5050 50  0001 C CNN
@@
 P 3400 2550
 AR Path="/652FE53F" Ref="C?"  Part="1"
-AR Path="/652C6908/652FE53F" Ref="C?"  Part="1"
-F 0 "C?" H 3300 2650 50  0000 L CNN
+AR Path="/652C6908/652FE53F" Ref="C101"  Part="1"
+F 0 "C101" V 3450 2300 50  0000 L CNN
 F 1 "2.2uF" V 3350 2300 50  0000 L CNN
 F 2 "" H 3438 2400 50  0001 C CNN
@@
 P 3400 2800
 AR Path="/652FE545" Ref="#PWR?"  Part="1"
-AR Path="/652C6908/652FE545" Ref="#PWR?"  Part="1"
-F 0 "#PWR?" H 3400 2550 50  0001 C CNN
+AR Path="/652C6908/652FE545" Ref="#PWR0101"  Part="1"
+F 0 "#PWR0101" H 3400 2550 50  0001 C CNN
 F 1 "GND" H 3405 2627 50  0000 C CNN
 F 2 "" H 3400 2800 50  0001 C CNN
@@
 L power:+3V3 #PWR?
 U 1 1 652FE54E
-P 3650 2950
+P 3850 2950
 AR Path="/652FE54E" Ref="#PWR?"  Part="1"
-AR Path="/652C6908/652FE54E" Ref="#PWR?"  Part="1"
-F 0 "#PWR?" H 3650 2800 50  0001 C CNN
-F 1 "+3V3" H 3665 3123 50  0000 C CNN
-F 2 "" H 3650 2950 50  0001 C CNN
-F 3 "" H 3650 2950 50  0001 C CNN
-	1    3650 2950
+AR Path="/652C6908/652FE54E" Ref="#PWR0102"  Part="1"
+F 0 "#PWR0102" H 3850 2800 50  0001 C CNN
+F 1 "+3V3" H 3865 3123 50  0000 C CNN
+F 2 "" H 3850 2950 50  0001 C CNN
+F 3 "" H 3850 2950 50  0001 C CNN
+	1    3850 2950
 	-1   0    0    1
 $EndComp
@@
 L Device:L_Core_Iron L?
 U 1 1 652FE554
-P 3650 2650
+P 3850 2650
 AR Path="/652FE554" Ref="L?"  Part="1"
-AR Path="/652C6908/652FE554" Ref="L?"  Part="1"
-F 0 "L?" H 3738 2696 50  0000 L CNN
-F 1 "10uH" H 3738 2605 50  0000 L CNN
-F 2 "" H 3650 2650 50  0001 C CNN
-F 3 "~" H 3650 2650 50  0001 C CNN
-	1    3650 2650
-	1    0    0    -1
-$EndComp
-Wire Wire Line
-	3650 2950 3650 2800
+AR Path="/652C6908/652FE554" Ref="L101"  Part="1"
+F 0 "L101" V 3800 2550 50  0000 L CNN
+F 1 "10uH" V 3950 2550 50  0000 L CNN
+F 2 "" H 3850 2650 50  0001 C CNN
+F 3 "~" H 3850 2650 50  0001 C CNN
+	1    3850 2650
+	1    0    0    -1
+$EndComp
+Wire Wire Line
+	3850 2950 3850 2800
 Wire Wire Line
 	3650 2500 3650 2400
@@
 	3400 2300 5000 2300
 Wire Wire Line
-	3650 2400 5000 2400
+	3650 2400 3850 2400
 Text HLabel 4400 2600 0    50   Input ~ 0
 PH0
@@
 Wire Wire Line
 	4400 3000 5000 3000
+Wire Wire Line
+	3850 2500 3850 2400
 Wire Bus Line
 	4600 3400 4600 5450
 Wire Bus Line
 	7450 3300 7450 5300
+Connection ~ 3850 2400
+Wire Wire Line
+	3850 2400 5000 2400
+Text HLabel 3650 2500 3    50   Input ~ 0
+VREF+
 $EndSCHEMATC

Commit message: updating sch. adding footprint for alps.
Parts:
- C101: footprint (none) -> Capacitor_SMD:C_0805_2012Metric_Pad1.18x1.45mm_HandSolder
- L101: footprint (none) -> Inductor_SMD:L_0805_2012Metric_Pad1.15x1.40mm_HandSolder
Changed lines of the file:
@@
 F 0 "C101" V 3450 2300 50  0000 L CNN
 F 1 "2.2uF" V 3350 2300 50  0000 L CNN
-F 2 "" H 3438 2400 50  0001 C CNN
+F 2 "Capacitor_SMD:C_0805_2012Metric_Pad1.18x1.45mm_HandSolder" H 3438 2400 50  0001 C CNN
 F 3 "~" H 3400 2550 50  0001 C CNN
 	1    3400 2550
@@
 F 0 "L101" V 3800 2550 50  0000 L CNN
 F 1 "10uH" V 3950 2550 50  0000 L CNN
-F 2 "" H 3850 2650 50  0001 C CNN
+F 2 "Inductor_SMD:L_0805_2012Metric_Pad1.15x1.40mm_HandSolder" H 3850 2650 50  0001 C CNN
 F 3 "~" H 3850 2650 50  0001 C CNN
 	1    3850 2650
@@
 Wire Wire Line
 	3850 2500 3850 2400
+Connection ~ 3850 2400
+Wire Wire Line
+	3850 2400 5000 2400
+Text HLabel 3650 2500 3    50   Input ~ 0
+VREF+
 Wire Bus Line
 	4600 3400 4600 5450
 Wire Bus Line
 	7450 3300 7450 5300
-Connection ~ 3850 2400
-Wire Wire Line
-	3850 2400 5000 2400
-Text HLabel 3650 2500 3    50   Input ~ 0
-VREF+
 $EndSCHEMATC
