File: apple_update/schematics/clock.sch (KiCad schematic (older format))
At the start: 3 parts, among them Y301 25MHZ 9PF

Commit message: updating sch. adding footprint for alps.
Parts:
- C301, C302: footprint (none) -> Capacitor_SMD:C_0805_2012Metric_Pad1.18x1.45mm_HandSolder
- Y301: footprint (none) -> Oscillator:Oscillator_SMD_Fordahl_DFAS15-4Pin_5.0x3.2mm_HandSoldering
Changed lines of the file:
@@
 F 0 "C302" H 5635 3654 50  0000 R CNN
 F 1 "12pF" H 5635 3745 50  0000 R CNN
-F 2 "" H 5788 3550 50  0001 C CNN
+F 2 "Capacitor_SMD:C_0805_2012Metric_Pad1.18x1.45mm_HandSolder" H 5788 3550 50  0001 C CNN
 F 3 "~" H 5750 3700 50  0001 C CNN
 	1    5750 3700
@@
 F 0 "Y301" H 5500 3718 50  0000 C CNN
 F 1 "25MHZ 9PF" V 5150 3500 50  0000 C CNN
-F 2 "" H 5500 3450 50  0001 C CNN
+F 2 "Oscillator:Oscillator_SMD_Fordahl_DFAS15-4Pin_5.0x3.2mm_HandSoldering" H 5500 3450 50  0001 C CNN
 F 3 "~" H 5500 3450 50  0001 C CNN
 	1    5500 3450
@@
 F 0 "C301" H 5185 3654 50  0000 R CNN
 F 1 "12pF" H 5185 3745 50  0000 R CNN
-F 2 "" H 5338 3550 50  0001 C CNN
+F 2 "Capacitor_SMD:C_0805_2012Metric_Pad1.18x1.45mm_HandSolder" H 5338 3550 50  0001 C CNN
 F 3 "~" H 5300 3700 50  0001 C CNN
 	1    5300 3700
