File: apple_update/schematics/power.sch (KiCad schematic (older format))
At the start: 12 parts, among them U601 ADP2108AUJ-3.3

Commit message: updating sch. adding footprint for alps.
Parts:
- C601, C602, C603, C604, C605, C606, C607, C608, C609: footprint (none) -> Capacitor_SMD:C_0805_2012Metric_Pad1.18x1.45mm_HandSolder
- L601: footprint (none) -> Inductor_SMD:L_0805_2012Metric_Pad1.15x1.40mm_HandSolder
Changed lines of the file:
@@
 F 0 "C605" V 6400 1900 50  0000 C CNN
 F 1 "100nF" V 6400 2100 50  0000 C CNN
-F 2 "" H 6388 1850 50  0001 C CNN
+F 2 "Capacitor_SMD:C_0805_2012Metric_Pad1.18x1.45mm_HandSolder" H 6388 1850 50  0001 C CNN
 F 3 "~" H 6350 2000 50  0001 C CNN
 	1    6350 2000
@@
 F 0 "C609" H 7415 4596 50  0000 L CNN
 F 1 "100nF" H 7415 4505 50  0000 L CNN
-F 2 "" H 7338 4400 50  0001 C CNN
+F 2 "Capacitor_SMD:C_0805_2012Metric_Pad1.18x1.45mm_HandSolder" H 7338 4400 50  0001 C CNN
 F 3 "~" H 7300 4550 50  0001 C CNN
 	1    7300 4550
@@
 F 0 "C607" H 6965 4596 50  0000 L CNN
 F 1 "100nF" H 6965 4505 50  0000 L CNN
-F 2 "" H 6888 4400 50  0001 C CNN
+F 2 "Capacitor_SMD:C_0805_2012Metric_Pad1.18x1.45mm_HandSolder" H 6888 4400 50  0001 C CNN
 F 3 "~" H 6850 4550 50  0001 C CNN
 	1    6850 4550
@@
 F 0 "C606" H 6515 4596 50  0000 L CNN
 F 1 "100nF" H 6515 4505 50  0000 L CNN
-F 2 "" H 6438 4400 50  0001 C CNN
+F 2 "Capacitor_SMD:C_0805_2012Metric_Pad1.18x1.45mm_HandSolder" H 6438 4400 50  0001 C CNN
 F 3 "~" H 6400 4550 50  0001 C CNN
 	1    6400 4550
@@
 F 0 "C604" H 6065 4596 50  0000 L CNN
 F 1 "100nF" H 6065 4505 50  0000 L CNN
-F 2 "" H 5988 4400 50  0001 C CNN
+F 2 "Capacitor_SMD:C_0805_2012Metric_Pad1.18x1.45mm_HandSolder" H 5988 4400 50  0001 C CNN
 F 3 "~" H 5950 4550 50  0001 C CNN
 	1    5950 4550
@@
 F 0 "C601" H 5115 4596 50  0000 L CNN
 F 1 "100nF" H 5115 4505 50  0000 L CNN
-F 2 "" H 5038 4400 50  0001 C CNN
+F 2 "Capacitor_SMD:C_0805_2012Metric_Pad1.18x1.45mm_HandSolder" H 5038 4400 50  0001 C CNN
 F 3 "~" H 5000 4550 50  0001 C CNN
 	1    5000 4550
@@
 F 0 "C603" H 5615 4596 50  0000 L CNN
 F 1 "100nF" H 5615 4505 50  0000 L CNN
-F 2 "" H 5538 4400 50  0001 C CNN
+F 2 "Capacitor_SMD:C_0805_2012Metric_Pad1.18x1.45mm_HandSolder" H 5538 4400 50  0001 C CNN
 F 3 "~" H 5500 4550 50  0001 C CNN
 	1    5500 4550
@@
 F 0 "C608" H 7015 3396 50  0000 L CNN
 F 1 "1.0uF" H 7015 3305 50  0000 L CNN
-F 2 "" H 6938 3200 50  0001 C CNN
+F 2 "Capacitor_SMD:C_0805_2012Metric_Pad1.18x1.45mm_HandSolder" H 6938 3200 50  0001 C CNN
 F 3 "~" H 6900 3350 50  0001 C CNN
 	1    6900 3350
@@
 F 0 "L601" V 6319 3200 50  0000 C CNN
 F 1 "1uH" V 6410 3200 50  0000 C CNN
-F 2 "" H 6500 3200 50  0001 C CNN
+F 2 "Inductor_SMD:L_0805_2012Metric_Pad1.15x1.40mm_HandSolder" H 6500 3200 50  0001 C CNN
 F 3 "~" H 6500 3200 50  0001 C CNN
 	1    6500 3200
@@
 F 0 "C602" H 5465 3546 50  0000 L CNN
 F 1 "1.0uF" H 5465 3455 50  0000 L CNN
-F 2 "" H 5388 3350 50  0001 C CNN
+F 2 "Capacitor_SMD:C_0805_2012Metric_Pad1.18x1.45mm_HandSolder" H 5388 3350 50  0001 C CNN
 F 3 "~" H 5350 3500 50  0001 C CNN
 	1    5350 3500
